File: Cartridge.sch (KiCad schematic (older format))
At the start: 3 parts, among them J1 Conn_01x32_Male, U1 AT28C256

Commit message: Add AT28C256 library
Parts:
- removed C1: 10nF, Capacitor_SMD:C_1206_3216Metric_Pad1.42x1.75mm_HandSolder, symbol Device:C
- removed J1: Conn_01x32_Male, Gameboy Cartridge:Edge Connector, symbol Connector:Conn_01x32_Male
- removed U1: AT28C256, Package_DIP:DIP-28_W15.24mm_Socket_LongPads, symbol Cartridge-rescue:AT28C256-Custom
Connections:
- no-connect marks 4 -> 0

Commit message: Update schematic to use new lib
Parts:
- added C?: 10n, symbol Device:C
- added J?: PAK_CONNECTOR, symbol Connector_Generic:Conn_01x32
- added U?: AT28C256-15PU, symbol AT28C256:AT28C256-15PU
Connections:
- new net: C?.1, J?.1 (Pin_1), U?.28 (VCC)
- new net: J?.10 (Pin_10), U?.6 (A4)
- new net: J?.11 (Pin_11), U?.5 (A5)
- new net: J?.12 (Pin_12), U?.4 (A6)
- new net: J?.13 (Pin_13), U?.3 (A7)
- new net: J?.14 (Pin_14), U?.25 (A8)
- new net: J?.15 (Pin_15), U?.24 (A9)
- new net: J?.16 (Pin_16), U?.21 (A10)
- new net: J?.17 (Pin_17), U?.23 (A11)
- new net: J?.18 (Pin_18), U?.2 (A12)
- new net: J?.19 (Pin_19), U?.26 (A13)
- new net: J?.20 (Pin_20), U?.1 (A14)
- new net: J?.22 (Pin_22), U?.11 (D0)
- new net: J?.23 (Pin_23), U?.12 (D1)
- new net: J?.24 (Pin_24), U?.13 (D2)
- new net: J?.25 (Pin_25), U?.15 (D3)
- new net: J?.26 (Pin_26), U?.16 (D4)
- new net: J?.27 (Pin_27), U?.17 (D5)
- new net: J?.28 (Pin_28), U?.18 (D6)
- new net: J?.29 (Pin_29), U?.19 (D7)
- new net: J?.3 (Pin_3), U?.27 (~WE)
- new net: C?.2, J?.32 (Pin_32), U?.14 (GND)
- new net: J?.4 (Pin_4), U?.22 (~OE)
- new net: J?.5 (Pin_5), U?.20 (~CE)
- new net: J?.6 (Pin_6), U?.10 (A0)
- new net: J?.7 (Pin_7), U?.9 (A1)
- new net: J?.8 (Pin_8), U?.8 (A2)
- new net: J?.9 (Pin_9), U?.7 (A3)
- no-connect marks 0 -> 4
Changed lines of the file:
@@
 Comment4 ""
 $EndDescr
+$Comp
+L Connector_Generic:Conn_01x32 J?
+U 1 1 5ED073BA
+P 4150 3450
+F 0 "J?" H 4150 5050 50  0000 C CNN
+F 1 "PAK_CONNECTOR" H 3900 1750 50  0000 C CNN
+F 2 "" H 4150 3450 50  0001 C CNN
+F 3 "~" H 4150 3450 50  0001 C CNN
+	1    4150 3450
+	-1   0    0    -1
+$EndComp
+$Comp
+L AT28C256:AT28C256-15PU U?
+U 1 1 5ED08DF2
+P 5200 3150
+F 0 "U?" H 5200 3150 50  0000 C CNN
+F 1 "AT28C256-15PU" H 5200 2350 50  0000 C CNN
+F 2 "" H 5200 3150 50  0001 C CNN
+F 3 "http://ww1.microchip.com/downloads/en/DeviceDoc/doc0006.pdf" H 5200 3150 50  0001 C CNN
+	1    5200 3150
+	1    0    0    -1
+$EndComp
+Wire Wire Line
+	4350 2450 4750 2450
+Wire Wire Line
+	4750 2550 4350 2550
+Wire Wire Line
+	4350 2650 4750 2650
+Wire Wire Line
+	4350 2750 4750 2750
+Wire Wire Line
+	4750 2850 4350 2850
+Wire Wire Line
+	4350 2950 4750 2950
+Wire Wire Line
+	4350 3050 4750 3050
+Wire Wire Line
+	4750 3150 4350 3150
+Wire Wire Line
+	4350 3250 4750 3250
+Wire Wire Line
+	4350 3350 4750 3350
+Wire Wire Line
+	4750 3450 4350 3450
+Wire Wire Line
+	4350 3550 4750 3550
+Wire Wire Line
+	4350 3650 4750 3650
+Wire Wire Line
+	4750 3750 4350 3750
+Wire Wire Line
+	4350 3850 4750 3850
+Wire Wire Line
+	5750 3850 5650 3850
+Wire Wire Line
+	5650 3750 5850 3750
+Wire Wire Line
+	5950 3650 5650 3650
+Wire Wire Line
+	5650 3550 6050 3550
+Wire Wire Line
+	5650 3450 6150 3450
+Wire Wire Line
+	5650 3350 6250 3350
+Wire Wire Line
+	5650 3250 6350 3250
+Wire Wire Line
+	5650 3150 6450 3150
+Wire Wire Line
+	4350 1950 5750 1950
+Wire Wire Line
+	5750 1950 5750 2450
+Wire Wire Line
+	5750 2450 5650 2450
+Wire Wire Line
+	5650 2550 6550 2550
+Wire Wire Line
+	6550 2550 6550 2400
+$Comp
+L Device:C C?
+U 1 1 5ED10C7E
+P 6550 2250
+F 0 "C?" H 6665 2296 50  0000 L CNN
+F 1 "10n" H 6665 2205 50  0000 L CNN
+F 2 "" H 6588 2100 50  0001 C CNN
+F 3 "~" H 6550 2250 50  0001 C CNN
+	1    6550 2250
+	1    0    0    -1
+$EndComp
+Wire Wire Line
+	6550 1950 5750 1950
+Wire Wire Line
+	6550 1950 6550 2100
+Connection ~ 5750 1950
+Wire Wire Line
+	6550 2550 6550 5050
+Wire Wire Line
+	6550 5050 4350 5050
+Connection ~ 6550 2550
+NoConn ~ 4350 4950
+NoConn ~ 4350 4850
+Wire Wire Line
+	4350 4350 6150 4350
+Wire Wire Line
+	4350 4250 6250 4250
+Wire Wire Line
+	4350 4150 6350 4150
+Wire Wire Line
+	4350 4050 6450 4050
+Wire Wire Line
+	4350 4450 6050 4450
+Wire Wire Line
+	4350 4550 5950 4550
+Wire Wire Line
+	4350 4650 5850 4650
+Wire Wire Line
+	4350 4750 5750 4750
+NoConn ~ 4350 3950
+Wire Wire Line
+	5750 3850 5750 4750
+Wire Wire Line
+	5850 3750 5850 4650
+Wire Wire Line
+	5950 3650 5950 4550
+Wire Wire Line
+	6050 3550 6050 4450
+Wire Wire Line
+	6150 3450 6150 4350
+Wire Wire Line
+	6250 3350 6250 4250
+Wire Wire Line
+	6350 3250 6350 4150
+Wire Wire Line
+	6450 3150 6450 4050
+NoConn ~ 4350 2050
+Wire Wire Line
+	5650 2950 6050 2950
+Wire Wire Line
+	6050 2950 6050 2350
+Wire Wire Line
+	6050 2350 4350 2350
+Wire Wire Line
+	5650 2750 5850 2750
+Wire Wire Line
+	5850 2750 5850 2150
+Wire Wire Line
+	5850 2150 4350 2150
+Wire Wire Line
+	4350 2250 5950 2250
+Wire Wire Line
+	5950 2250 5950 2850
+Wire Wire Line
+	5950 2850 5650 2850
 $EndSCHEMATC
